File: PCB/80% Keyboard.kicad_pcb (KiCad board)
At the start: 2 copper layers, 359 x 136.7 mm, 201 parts, among them J1 USB_C_Receptacle_USB2.0_16P, SW1 Esc, SW10 A, SW102 Right, SW11 Z, SW12 Win, SW13 F2, SW14 2, SW15 W, SW16 S, SW17 X, SW18 Alt, SW19 F3, SW2 Tilde ~, SW20 3, SW21 E, SW22 D, SW23 C, SW24 RotaryEncoder, SW25 F4, SW26 4, SW27 R, SW28 F, SW29 V, SW3 Tab, SW30 SW_BOOT, SW31 F5, SW32 5, SW33 T, SW34 G, SW35 B, SW36 Space, SW37 F6, SW38 6, SW39 Y, SW4 CapsLock, SW40 H, SW41 N, SW42 SW_RESET, SW43 F7, SW44 7, SW45 U, SW46 J, SW47 M, SW49 F8, SW5 Shift, SW50 8, SW51 I, SW52 K, SW53 Comma, SW54 R_Alt, SW55 F9, SW56 9, SW57 O, SW58 L, SW59 Full Stop, SW6 Ctrl, SW60 R_Win, SW61 F10, SW62 0, SW63 P, SW64 Semicolon, SW65 F Slash, SW66 Fn, SW67 F11, SW68 Minus -, SW69 [, SW7 F1, SW70 Apostrophe, SW71 R_Shift, SW72 R_Ctrl, SW73 F12, SW74 Plus +, SW75 ], SW76 Enter, SW8 1, SW80 Backspace, SW81 B Slash, SW85 PrtSc, SW86 Insert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

Commit message: Artwork + Name + Journal
Parts:
- added G***: LOGO, LOGO, F.Cu at (370.0, 146.0)
- added G***: LOGO, LOGO, B.Cu at (370.0, 146.0)
- added H1: M2, MountingHole:MountingHole_2.2mm_M2, F.Cu at (55.0, 95.0)
- added H2: M2, MountingHole:MountingHole_2.2mm_M2, F.Cu at (298.0, 95.0)
- added H3: M2, MountingHole:MountingHole_2.2mm_M2, F.Cu at (81.0, 195.0)
- added H4: M2, MountingHole:MountingHole_2.2mm_M2, F.Cu at (272.0, 195.0)
- added H5: M2, MountingHole:MountingHole_2.2mm_M2, F.Cu at (362.0, 95.0)
- added H6: M2, MountingHole:MountingHole_2.2mm_M2, F.Cu at (362.0, 195.0)
Routing:
- net GND: track 680.2 -> 675.9 mm
Other:
- board size 359 x 136.7 mm -> 359 x 137 mm
- board text added: "Made by Xavier :3"

Commit message: All of CAD Case + Clean Up of PCB Files
Parts:
- removed H1, H2, H3, H4, H5, H6: M2, MountingHole:MountingHole_2.2mm_M2
- D1, D10, D102, D11, D12, D13, D14, D15, D16, D17, D18, D19, D2, D20, D21, D22, D23, D25, D26, D27, D28, D29, D3, D31, D32, D33, D34, D35, D36, D37, D38, D39, D4, D40, D41, D43, D44, D45, D46, D47, D49, D5, D50, D51, D52, D53, D54, D55, D56, D57, D58, D59, D6, D60, D61, D62, D63, D64, D65, D66, D67, D68, D69, D7, D70, D71, D72, D73, D74, D75, D76, D8, D80, D81, D85, D86, D87, D9, D90, D91, D92, D93, D95, D96, D97, D98, D99, SW1, SW10, SW102, SW11, SW12, SW13, SW14, SW15, SW16, SW17, SW18, SW19, SW2, SW20, SW21, SW22, SW23, SW25, SW26, SW27, SW28, SW29, SW3, SW31, SW32, SW33, SW34, SW35, SW36, SW37, SW38, SW39, SW4, SW40, SW41, SW43, SW44, SW45, SW46, SW47, SW49, SW5, SW50, SW51, SW52, SW53, SW54, SW55, SW56, SW57, SW58, SW59, SW6, SW60, SW61, SW62, SW63, SW64, SW65, SW66, SW67, SW68, SW69, SW7, SW70, SW71, SW72, SW73, SW74, SW75, SW76, SW8, SW80, SW81, SW85, SW86, SW87, SW9, SW90, SW91, SW92, SW93, SW95, SW96, SW97, SW98, SW99: moved to B.Cu
- moved D36 114.3 mm to (221.7, 178.0), turned to 180 degrees
- moved D5 38.1 mm to (74.1, 159.0), turned to 180 degrees
- moved D71 31.1 mm to (300.5, 159.0), turned to 180 degrees
- moved D4 28.6 mm to (64.6, 139.9), turned to 180 degrees
- moved D76 26.6 mm to (305.5, 139.9), turned to 180 degrees
- moved D80 24.0 mm to (307.6, 101.8), turned to 180 degrees
- moved D3 23.8 mm to (59.8, 120.9), turned to 180 degrees
- moved D54 19.1 mm to (245.6, 178.0), turned to 180 degrees
- moved D60 19.1 mm to (269.4, 178.0), turned to 180 degrees
- moved D66 19.1 mm to (293.2, 178.0), turned to 180 degrees
- moved D12 19.0 mm to (78.9, 178.0), turned to 180 degrees
- moved D18 19.0 mm to (102.7, 178.0), turned to 180 degrees
- moved D6 19.0 mm to (55.0, 178.0), turned to 180 degrees
- moved D72 14.9 mm to (312.9, 178.0), turned to 180 degrees
- moved D7 14.3 mm to (74.1, 78.6), turned to 180 degrees
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Routing:
- net /ROW3: track 307.9 -> 276.2 mm, vias 0 -> 1
- net /COL0: track 446.8 -> 468.5 mm, vias 12 -> 1
- net /ROW4: track 345.8 -> 324.5 mm, vias 0 -> 2
- net /COL11: track 205.4 -> 221.8 mm, vias 12 -> 11
- net /COL14: track 206.3 -> 222.3 mm, vias 7 -> 8
- net /COL12: track 133.0 -> 147.9 mm, vias 8 -> 7
- net GND: track 675.9 -> 690.7 mm
- net Net-(D71-A): track 18.2 -> 4.51 mm
- net /COL13: track 89.9 -> 102.0 mm, vias 4 -> 3
- net /COL16: track 186.9 -> 175.8 mm, vias 2 -> 8
- net /USB_DM: track 337.9 -> 348.5 mm
- net /ROW2: track 378.2 -> 367.9 mm
- net /USB_DP: track 337.0 -> 346.1 mm
- net Net-(D76-A): track 13.4 -> 4.47 mm
- net /ROW5: track 383.9 -> 392.4 mm, vias 2 -> 3
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Other:
- board size 359 x 137 mm -> 353 x 135 mm
- board text removed: "Made by Xavier :3"

Commit message: Bom Stuff
Parts:
- U1: footprint Package_SO:SOIC-8_3.9x4.9mm_P1.27mm -> Package_SO:SOIC-8_5.3x5.3mm_P1.27mm
Routing:
- net /QSPI_SD1: track 35.4 -> 33.6 mm
- net /QSPI_SCLK: track 22.3 -> 21.2 mm
- net /QSPI_SD2: track 37.6 -> 36.5 mm
- net /QSPI_SD3: track 20.0 -> 18.9 mm
- net /QSPI_SD0: track 23.1 -> 22.0 mm
- net /3V3: track 388.6 -> 387.6 mm
